Commit message: 完成urdf实例

File: src/lesson7_urdf/urdf/sai_robot.urdf (robot description, URDF)
Before this commit: robot saibot, 1 links, 0 joints
Links:
- added link back_caster_link; visual sphere radius=0.015
- added link camera_link; visual box size=0.03 0.04 0.04
- added link front_caster_link; visual sphere radius=0.015
- added link kinect_link; visual mesh filename=package://lesson7_urdf/meshes/kinect.dae
- added link laser_link; visual cylinder length=0.06 radius=0.05
- added link left_wheel_link; visual cylinder length=0.025 radius=0.06
- added link right_wheel_link; visual cylinder length=0.025 radius=0.06
Joints:
- added joint back_caster_joint: type continuous, parent base_link, child back_caster_link, origin xyz=-0.18 0.0 -0.095 rpy=0.0 0.0 0.0, axis 0.0 1.0 0.0
- added joint camera_joint: type fixed, parent base_link, child camera_link, origin xyz=0.17 0.0 0.1 rpy=0.0 0.0 0.0
- added joint front_caster_joint: type continuous, parent base_link, child front_caster_link, origin xyz=0.18 0.0 -0.095 rpy=0.0 0.0 0.0, axis 0.0 1.0 0.0
- added joint kinect_joint: type fixed, parent base_link, child kinect_link, origin xyz=-0.17 0.0 0.115 rpy=0.0 0.0 -1.57
- added joint laser_joint: type fixed, parent base_link, child laser_link, origin xyz=0.0 0.0 0.106 rpy=0.0 0.0 0.0
- added joint left_wheel_joint: type continuous, parent base_link, child left_wheel_link, origin xyz=0.0 0.19 -0.05 rpy=0.0 0.0 0.0, axis 0.0 1.0 0.0
- added joint right_wheel_joint: type continuous, parent base_link, child right_wheel_link, origin xyz=0.0 -0.19 -0.05 rpy=0.0 0.0 0.0, axis 0.0 1.0 0.0
