Commit message: 解决kinect方向的问题

File: src/lesson11_gazebo/urdf/sai_robot.urdf.xacro (robot description, xacro)
@@ -247,5 +247,5 @@
     </gazebo>
     <joint name="kinect_joint" type="fixed">
-        <origin xyz="-${camera_x} 0.0 0.115" rpy="0.0 0.0 -${M_PI / 2}"/>
+        <origin xyz="-${camera_x} 0.0 0.115" rpy="0.0 0.0 -${M_PI}"/>
         <parent link="base_link"/>
         <child link="kinect_link"/>
@@ -253,5 +253,5 @@
     <link name="kinect_link">
         <visual>
-            <origin xyz="0.0 0.0 0.0" rpy="0.0 0.0 0.0"/>
+            <origin xyz="0.0 0.0 0.0" rpy="0.0 0.0 ${M_PI / 2}"/>
             <geometry>
                 <!-- Load texture description file -->
@@ -326,5 +326,5 @@
             <update_rate>20</update_rate>
             <camera>
-                <horizontal_fov>${60 * M_PI / 180}</horizontal_fov>
+                <horizontal_fov>1.57</horizontal_fov>
                 <image>
                     <width>640</width>
@@ -336,9 +336,4 @@
                     <far>8</far>
                 </clip>
-                <noise>
-                    <type>gaussian</type>
-                    <mean>0.0</mean>
-                    <stddev>0.007</stddev>
-                </noise>
             </camera>
             <plugin name="gazebo_kinect" filename="libgazebo_ros_openni_kinect.so">

Commit message: 完成Gazebo仿真环境

File: src/lesson11_gazebo/urdf/sai_robot.urdf.xacro (robot description, xacro)
@@ -13,8 +13,9 @@
     <xacro:property name="wheel_y" value="0.19" />
     <!-- 支撑轮的半径、x轴 -->
-    <xacro:property name="caster_mass" value="0.5" />
+    <xacro:property name="caster_mass" value="0.1" />
     <xacro:property name="caster_radius" value="0.015" />
     <xacro:property name="caster_x" value="0.18" />
     <!-- 摄像头的的长、宽、高、x轴 -->
+    <xacro:property name="camera_mass" value="0.1" />
     <xacro:property name="camera_x" value="0.17" />
     <xacro:property name="camera_length" value="0.03" />
@@ -22,6 +23,7 @@
     <xacro:property name="camera_high" value="0.04" />
     <!-- 激光雷达头的的半径和高度 -->
+    <xacro:property name="laser_mass" value="0.1" />
     <xacro:property name="laser_radius" value="0.05" />
-    <xacro:property name="laser_length" value="0.06" />
+    <xacro:property name="laser_length" value="0.15" />
     <!-- 球形的惯性矩阵 -->
     <xacro:macro name="sphere_inertial_matrix" params="m r">
@@ -36,4 +38,11 @@
             <mass value="${m}"/>
             <inertia ixx="${m * (3 * r * r + h * h) / 12}" ixy="0.0" ixz="0.0" iyy="${m * (3 * r * r + h * h) / 12}" iyz="0.0" izz="${m * r * r / 2}"/>
+        </inertial>
+    </xacro:macro>
+    <!-- 立方体的惯性矩阵 -->
+    <xacro:macro name="box_inertial_matrix" params="m">
+        <inertial>
+            <mass value="${m}"/>
+            <inertia ixx="${m}" ixy="0.0" ixz="0.0" iyy="${m}" iyz="0.0" izz="${m}"/>
         </inertial>
     </xacro:macro>
@@ -219,4 +228,5 @@
             </geometry>
         </collision>
+        <box_inertial_matrix m="${camera_mass}" />
     </link>
     <gazebo reference="camera_link">
@@ -242,4 +252,5 @@
             </geometry>
         </collision>
+        <cylinder_inertial_matrix m="${laser_mass}" r="${laser_radius}" h="${laser_length}" />
     </link>
     <gazebo reference="laser_link">
@@ -285,4 +296,5 @@
         </plugin>
     </gazebo>
+    <!-- add Gazebo Camera -->
     <gazebo reference="camera_link">
         <sensor type="camera" name="camera_node">
@@ -321,4 +333,5 @@
         </sensor>
     </gazebo>
+    <!-- add Gazebo Kinect -->
     <gazebo reference="kinect_link">
         <sensor type="depth" name="kinect_node">
@@ -357,4 +370,5 @@
         </sensor>
     </gazebo>
+    <!-- add Gazebo Laser -->
     <gazebo reference="laser_link">
         <sensor type="ray" name="laser_node">
@@ -368,5 +382,5 @@
                         <resolution>1</resolution>
                         <min_angle>-3</min_angle>
-                        <max_angle>-3</max_angle>
+                        <max_angle>3</max_angle>
                     </horizontal>
                 </scan>
